Commit message: moveit

File: src/robo1_description/urdf/modified_test1.urdf (robot description, URDF)
Before this commit: robot test_1, 24 links, 23 joints
Links:
- link LewanSoul_LX-16A_1: geometry collision mesh filename=file://$(find robo1_description)/meshes/LewanSoul_LX-16A_1.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; visual mesh filename=file://$(find robo1_description)/meshes/LewanSoul_LX-16A_1.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
- link LewanSoul_LX-16A_2: geometry collision mesh filename=file://$(find robo1_description)/meshes/LewanSoul_LX-16A_2.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; visual mesh filename=file://$(find robo1_description)/meshes/LewanSoul_LX-16A_2.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
- link LewanSoul_LX-16A_3: geometry collision mesh filename=file://$(find robo1_description)/meshes/LewanSoul_LX-16A_3.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; visual mesh filename=file://$(find robo1_description)/meshes/LewanSoul_LX-16A_3.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
- link LewanSoul_LX-16A_4: geometry collision mesh filename=file://$(find robo1_description)/meshes/LewanSoul_LX-16A_4.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; visual mesh filename=file://$(find robo1_description)/meshes/LewanSoul_LX-16A_4.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
- link LewanSoul_LX-16A_5: geometry collision mesh filename=file://$(find robo1_description)/meshes/LewanSoul_LX-16A_5.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; visual mesh filename=file://$(find robo1_description)/meshes/LewanSoul_LX-16A_5.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
- link LewanSoul_LX-16A_6: geometry collision mesh filename=file://$(find robo1_description)/meshes/LewanSoul_LX-16A_6.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; visual mesh filename=file://$(find robo1_description)/meshes/LewanSoul_LX-16A_6.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
- link LewanSoul_LX-16A_7: geometry collision mesh filename=file://$(find robo1_description)/meshes/LewanSoul_LX-16A_7.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; visual mesh filename=file://$(find robo1_description)/meshes/LewanSoul_LX-16A_7.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
- link LewanSoul_LX-16A_8: geometry collision mesh filename=file://$(find robo1_description)/meshes/LewanSoul_LX-16A_8.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; visual mesh filename=file://$(find robo1_description)/meshes/LewanSoul_LX-16A_8.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
- link ankleL_1: geometry collision mesh filename=file://$(find robo1_description)/meshes/ankleL_1.stl; visual mesh filename=file://$(find robo1_description)/meshes/ankleL_1.stl
- link ankleL_2: geometry collision mesh filename=file://$(find robo1_description)/meshes/ankleL_2.stl; visual mesh filename=file://$(find robo1_description)/meshes/ankleL_2.stl
- link base_link: geometry collision mesh filename=file://$(find robo1_description)/meshes/base_v2_v1_1.stl; visual mesh filename=file://$(find robo1_description)/meshes/base_v2_v1_1.stl
- link batteryHolder_v2_1: geometry collision mesh filename=file://$(find robo1_description)/meshes/batteryHolder_v2_1.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; visual mesh filename=file://$(find robo1_description)/meshes/batteryHolder_v2_1.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
- link flankL_1: geometry collision mesh filename=file://$(find robo1_description)/meshes/flankL_1.stl; visual mesh filename=file://$(find robo1_description)/meshes/flankL_1.stl
- link flankR_1: geometry collision mesh filename=file://$(find robo1_description)/meshes/flankR_1.stl; visual mesh filename=file://$(find robo1_description)/meshes/flankR_1.stl
- link footL_1: geometry collision mesh filename=file://$(find robo1_description)/meshes/footL_1.stl; visual mesh filename=file://$(find robo1_description)/meshes/footL_1.stl
- link footR_1: geometry collision mesh filename=file://$(find robo1_description)/meshes/footR_1.stl; visual mesh filename=file://$(find robo1_description)/meshes/footR_1.stl
- link hip_1: geometry collision mesh filename=file://$(find robo1_description)/meshes/hip_1.stl; visual mesh filename=file://$(find robo1_description)/meshes/hip_1.stl
- link hip_2: geometry collision mesh filename=file://$(find robo1_description)/meshes/hip_2.stl; visual mesh filename=file://$(find robo1_description)/meshes/hip_2.stl
- link leg_segment_1: geometry collision mesh filename=file://$(find robo1_description)/meshes/leg_segment_1.stl; visual mesh filename=file://$(find robo1_description)/meshes/leg_segment_1.stl
- link leg_segment_2: geometry collision mesh filename=file://$(find robo1_description)/meshes/leg_segment_2.stl; visual mesh filename=file://$(find robo1_description)/meshes/leg_segment_2.stl
- link leg_segment_3: geometry collision mesh filename=file://$(find robo1_description)/meshes/leg_segment_3.stl; visual mesh filename=file://$(find robo1_description)/meshes/leg_segment_3.stl
- link leg_segment_4: geometry collision mesh filename=file://$(find robo1_description)/meshes/leg_segment_4.stl; visual mesh filename=file://$(find robo1_description)/meshes/leg_segment_4.stl
- link motors_1: geometry collision mesh filename=file://$(find robo1_description)/meshes/motors_1.stl scale=0.001 0.001 0.001; visual mesh filename=file://$(find robo1_description)/meshes/motors_1.stl scale=0.001 0.001 0.001
