Commit message: working ros_control

File: src/robo1_description/urdf/test_1.ros2_control.xacro (robot description, xacro)
@@ -1,7 +1,5 @@
 <?xml version="1.0"?>
 <robot xmlns:xacro="http://www.ros.org/wiki/xacro">
-    <xacro:macro name="test_1_ros2_control" params="name initial_positions_file">
-        <xacro:property name="initial_positions" value="${xacro.load_yaml(initial_positions_file)['initial_positions']}"/>
-        <ros2_control name="${name}" type="system">
+        <ros2_control name="legs" type="system">
             <hardware>
                 <!-- By default, set up controllers for simulation. This won't work on real hardware -->
@@ -11,5 +9,5 @@
                 <command_interface name="position"/>
                 <state_interface name="position">
-                  <param name="initial_value">${initial_positions['Revolute_5_1']}</param>
+                  <param name="initial_value">0.0</param>
                 </state_interface>
             </joint>
@@ -17,5 +15,5 @@
                 <command_interface name="position"/>
                 <state_interface name="position">
-                  <param name="initial_value">${initial_positions['Revolute_3_1']}</param>
+                  <param name="initial_value">0.0</param>
                 </state_interface>
             </joint>
@@ -23,5 +21,5 @@
                 <command_interface name="position"/>
                 <state_interface name="position">
-                  <param name="initial_value">${initial_positions['Fastened_5_1']}</param>
+                  <param name="initial_value">0.0</param>
                 </state_interface>
             </joint>
@@ -29,5 +27,5 @@
                 <command_interface name="position"/>
                 <state_interface name="position">
-                  <param name="initial_value">${initial_positions['Revolute_7']}</param>
+                  <param name="initial_value">0.0</param>
                 </state_interface>
             </joint>
@@ -35,5 +33,5 @@
                 <command_interface name="position"/>
                 <state_interface name="position">
-                  <param name="initial_value">${initial_positions['Revolute_5']}</param>
+                  <param name="initial_value">0.0</param>
                 </state_interface>
             </joint>
@@ -41,5 +39,5 @@
                 <command_interface name="position"/>
                 <state_interface name="position">
-                  <param name="initial_value">${initial_positions['Revolute_3']}</param>
+                  <param name="initial_value">0.0</param>
                 </state_interface>
             </joint>
@@ -47,5 +45,5 @@
                 <command_interface name="position"/>
                 <state_interface name="position">
-                  <param name="initial_value">${initial_positions['Revolute_2']}</param>
+                  <param name="initial_value">0.0</param>
                 </state_interface>
             </joint>
@@ -53,8 +51,7 @@
                 <command_interface name="position"/>
                 <state_interface name="position">
-                  <param name="initial_value">${initial_positions['Revolute_1']}</param>
+                  <param name="initial_value">0.0</param>
                 </state_interface>
             </joint>
         </ros2_control>
-    </xacro:macro>
 </robot>
